File: H03R00-T/Design/H03R00-T.brd (EAGLE design)
At the start: 34.6 x 30 mm, 10 parts, among them P1 HEXABIT_17.32_POWER_ONLY, P2 VCC, U1 LM2575SX-3.3/NOPB

Commit message: Update H03R00-T
Add -T extension to terminal block version
Update schematics and fix VDD connection
Regenerate output
Connections:
- removed net OUT: C2.1, L1.2, U1.4
- net VDD: now also C2.1, L1.2, U1.4
Routing:
- net VDD: track 87.2 -> 106.6 mm, vias 0 -> 1
- net OUT: track 19.4 -> 0.00 mm, vias 1 -> 0
Changed lines of the file:
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@@
 <drawing>
 <settings>
-<setting alwaysvectorfont="no"/>
+<setting alwaysvectorfont="yes"/>
 <setting verticaltext="up"/>
 </settings>
@@
 <wire x1="26.3602" y1="20.3102" x2="42.8802" y2="20.3102" width="0.3048" layer="1"/>
 <wire x1="42.8802" y1="20.3102" x2="51.1402" y2="34.6202" width="0.3048" layer="1"/>
+<contactref element="L1" pad="2"/>
+<contactref element="C2" pad="1"/>
+<contactref element="U1" pad="4"/>
+<wire x1="24.765" y1="38.71" x2="24.765" y2="39.726871875" width="1.016" layer="16"/>
+<wire x1="24.765" y1="39.726871875" x2="26.330909375" y2="41.29278125" width="1.016" layer="16"/>
+<via x="26.330909375" y="41.29278125" extent="1-16" drill="0.35"/>
+<wire x1="26.330909375" y1="41.29278125" x2="26.348690625" y2="41.275" width="0.3048" layer="1"/>
+<wire x1="26.348690625" y1="41.275" x2="29.567" y2="41.275" width="1.016" layer="1"/>
+<wire x1="31.69158125" y1="34.946590625" x2="32.8422" y2="33.795971875" width="1.016" layer="16"/>
+<wire x1="31.69158125" y1="34.946590625" x2="26.615390625" y2="34.946590625" width="1.016" layer="16"/>
+<wire x1="24.765" y1="36.79698125" x2="24.765" y2="38.71" width="1.016" layer="16"/>
+<wire x1="26.615390625" y1="34.946590625" x2="24.765" y2="36.79698125" width="1.016" layer="16"/>
+<wire x1="32.8422" y1="33.795971875" x2="32.8422" y2="32.1056" width="1.016" layer="16"/>
 </signal>
 <signal name="N$1">
@@
 <wire x1="24.767909375" y1="35.775" x2="23.114" y2="35.775" width="1.016" layer="1"/>
 </signal>
-<signal name="OUT">
-<contactref element="L1" pad="2"/>
-<contactref element="C2" pad="1"/>
-<contactref element="U1" pad="4"/>
-<wire x1="24.765" y1="38.71" x2="24.765" y2="39.726871875" width="1.016" layer="16"/>
-<wire x1="24.765" y1="39.726871875" x2="26.330909375" y2="41.29278125" width="1.016" layer="16"/>
-<via x="26.330909375" y="41.29278125" extent="1-16" drill="0.35"/>
-<wire x1="26.330909375" y1="41.29278125" x2="26.348690625" y2="41.275" width="0.3048" layer="1"/>
-<wire x1="26.348690625" y1="41.275" x2="29.567" y2="41.275" width="1.016" layer="1"/>
-<wire x1="31.69158125" y1="34.946590625" x2="32.8422" y2="33.795971875" width="1.016" layer="16"/>
-<wire x1="31.69158125" y1="34.946590625" x2="26.615390625" y2="34.946590625" width="1.016" layer="16"/>
-<wire x1="24.765" y1="36.79698125" x2="24.765" y2="38.71" width="1.016" layer="16"/>
-<wire x1="26.615390625" y1="34.946590625" x2="24.765" y2="36.79698125" width="1.016" layer="16"/>
-<wire x1="32.8422" y1="33.795971875" x2="32.8422" y2="32.1056" width="1.016" layer="16"/>
-</signal>
 </signals>
