File: H03R00-T/Design/H03R00-T.sch (EAGLE design)
At the start: 10 parts, among them P1 HEXABIT_17.32_POWER_ONLY, P2 VCC, U1 LM2575SX-3.3/NOPB

Commit message: Update H03R00-T
Add -T extension to terminal block version
Update schematics and fix VDD connection
Regenerate output
Connections:
- removed net OUT: C2.+, L1.2, U1.FB
- net VDD: now also C2.+, L1.2, U1.FB
Other:
- note added: "3.3V/1A DC-DC Buck Power Supply w/ Terminal Block"
- note added: "H03R00-T"
- note added: "VCC=5-40 Volts"
- note removed: "3.3V/1A DC-DC Buck Power Supply"
- note removed: "H03R0"
- moved on the sheet: C1, C2, D1, D2, J, L1, P1, P2, R1, U1
