File: H03R0-J/Design/H03R0-J.sch (EAGLE design)
At the start: 10 parts, among them J1 0.0R, P1 HEXABIT_17.32_POWER_ONLY, P2 VCC, U1 LM2575SX-3.3/NOPB

Commit message: -Standarize the files and folders
Other:
- note added: "H03R0-J"
- note added: "H03R0-J_Frontend"
- note removed: "Anas Kaadan"
- note removed: "H03R00-J"
- note removed: "H03R0_Frontend"
Changed lines of the file:
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@@
 <?xml version="1.0" encoding="utf-8"?>
 <!DOCTYPE eagle SYSTEM "eagle.dtd">
-<eagle version="9.3.0">
+<eagle version="9.6.2">
 <drawing>
 <settings>
-<setting alwaysvectorfont="yes"/>
+<setting alwaysvectorfont="no"/>
 <setting verticaltext="up"/>
 </settings>
@@
 <text x="215.9" y="5.3848" size="1.9304" layer="100" font="vector">Sheet   of</text>
 <text x="199.4662" y="19.6342" size="1.9304" layer="100" font="vector">Title</text>
-<text x="180.9242" y="19.6342" size="1.9304" layer="102" font="vector">H03R00-J</text>
+<text x="180.9242" y="19.6342" size="1.9304" layer="102" font="vector">H03R0-J</text>
 <text x="192.0078" y="11.7914" size="1.6764" layer="101" font="vector" align="center">3.3V/1A DC-DC Buck Power Supply
 w/ Barrel Jack</text>
-<text x="206.3242" y="19.6342" size="1.9304" layer="101" font="vector">H03R0_Frontend</text>
+<text x="206.3242" y="19.6342" size="1.9304" layer="101" font="vector">H03R0-J_Frontend</text>
 <wire x1="168.91" y1="3.81" x2="168.91" y2="8.128" width="0.1524" layer="205"/>
 <wire x1="168.91" y1="8.128" x2="168.91" y2="18.288" width="0.1524" layer="205"/>
@@
 <wire x1="231.14" y1="18.288" x2="231.14" y2="22.86" width="0.1524" layer="205"/>
 <text x="242.6462" y="6.1722" size="1.9304" layer="100" font="vector">www.hexabitz.com</text>
-<text x="180.4178" y="4.9414" size="1.9304" layer="101" font="vector">Anas Kaadan</text>
 <text x="20.32" y="198.12" size="1.778" layer="150">VDD=3.3 Volts</text>
 <text x="20.32" y="198.12" size="1.778" layer="150">VDD=3.3 Volts</text>
